Commit message: changed_the_bot_dimensions_needed_ones

File: install/model_py/share/model_py/urdf/robot_core.urdf.xacro (robot description, xacro)
@@ -35,5 +35,5 @@
             <origin xyz="0.135 0 0.052885"/>
             <geometry>
-                <box size="0.27 0.168 0.10577"/>
+                <box size="1.5 1 0.6"/>
             </geometry>
             <material name="white"/>
@@ -42,8 +42,8 @@
             <origin xyz="0.135 0 0.052885"/>
             <geometry>
-                <box size="0.27 0.168 0.10577"/>
+                <box size="1.5 1 0.6"/>
             </geometry>
         </collision>
-        <xacro:inertial_box mass="0.750" x="0.27" y="0.168" z="0.10577">
+        <xacro:inertial_box mass="70" x="0.27" y="0.168" z="0.10577">
             <origin xyz="0.135 0 0.052885" rpy="0 0 0"/>
         </xacro:inertial_box>
@@ -56,5 +56,5 @@
         <parent link="base_link"/>
         <child link="left_wheel"/>
-        <origin xyz="0.12 0.0965 0" rpy="-${pi/2} 0 0"/>  <!-- we are rotating the whole bot 90 degrees wrt x axis..-->
+        <origin xyz="0.3 0.4 -0.25" rpy="-${pi/2} 0 0"/>  <!-- we are rotating the whole bot 90 degrees wrt x axis..-->
         <axis xyz="0 0 1"/>
     </joint>
@@ -62,5 +62,5 @@
         <visual>
             <geometry>
-                <cylinder radius="0.04" length="0.025"/>
+                <cylinder radius="0.25" length="0.130"/>
             </geometry>
             <material name="black"/>
@@ -68,8 +68,8 @@
         <collision>
             <geometry>
-                <sphere radius="0.04"/>
+                <sphere radius="0.25"/>
             </geometry>
         </collision>
-        <xacro:inertial_cylinder mass="0.1" length="0.025" radius="0.04">
+        <xacro:inertial_cylinder mass="3" length="0.130" radius="0.25">
             <origin xyz = "0 0 0" rpy = "0 0 0 "/>
         </xacro:inertial_cylinder>
@@ -82,5 +82,5 @@
         <parent link="base_link"/>
         <child link="right_wheel"/>
-        <origin xyz="0.12 -0.0965 0" rpy="${pi/2} 0 0"/>  <!-- we are rotating the whole bot 90 degrees wrt x axis..-->
+        <origin xyz="0.3 -0.4 -0.25" rpy="${pi/2} 0 0"/>  <!-- we are rotating the whole bot 90 degrees wrt x axis..-->
         <axis xyz="0 0 -1"/>
     </joint>
@@ -88,5 +88,5 @@
         <visual>
             <geometry>
-                <cylinder radius="0.04" length="0.025"/>
+                <cylinder radius="0.25" length="0.130"/>
             </geometry>
             <material name="black"/>
@@ -94,9 +94,9 @@
         <collision>
             <geometry>
-                <sphere radius="0.04"/>
+                <sphere radius="0.25"/>
             </geometry>
             <material name="black"/>
         </collision>
-        <xacro:inertial_cylinder mass="0.1" length="0.025" radius="0.04">
+        <xacro:inertial_cylinder mass="3" length="0.130" radius="0.25">
             <origin xyz = "0 0 0" rpy = "0 0 0 "/>
         </xacro:inertial_cylinder>
@@ -109,20 +109,20 @@
         <parent link="chassis"/>
         <child link="caster_wheel_left"/>
-        <origin xyz="0.035 0 0"/>
+        <origin xyz="-0.35 0 -0.3"/>
     </joint>
     <link name="caster_wheel_left">
         <visual>
             <geometry>
-                <sphere radius="0.04"/>
+                <sphere radius="0.2"/>
             </geometry>
-            <material name="orange"/>
+            <material name="black"/>
         </visual>
         <collision>
             <geometry>
-                <sphere radius="0.04"/>
+                <sphere radius="0.2"/>
             </geometry>
-            <material name="orange"/>
+            <material name="black"/>
         </collision>
-        <xacro:inertial_sphere mass="0.05" radius="0.04">
+        <xacro:inertial_sphere mass="1" radius="0.2">
             <origin xyz="0 0 0" rpy="0 0 0"/>
         </xacro:inertial_sphere>

File: install/model_py/share/model_py/urdf/run.urdf.xacro (robot description, xacro)
@@ -3,5 +3,6 @@
     <!-- <xacro:arg name="use_ros2_control" default="true"/> -->
     <xacro:include filename="robot_core.urdf.xacro" />
-    <xacro:include filename="lidar.urdf.xacro" />
+    <xacro:include filename="gazebo_control.xacro" />
+    <!-- <xacro:include filename="lidar.urdf.xacro" /> -->
     <!-- <xacro:if value="$(arg use_ros2_control)">
         <xacro:include filename="ros2_control.xacro" />
