Commit message: commit

File: install/model_py/share/model_py/urdf/lidar.urdf.xacro (robot description, xacro)
@@ -1,52 +1,67 @@
 <?xml version="1.0"?>
-<robot xmlns:xacro="http://www.ros.org/wiki/xacro" >
-    <joint name="laser_joint" type="fixed">
-        <parent link="chassis"/>
-        <child link="laser_frame"/>
-        <origin xyz="0.215 0 0.11" rpy="0 0 0"/>
-    </joint>
-    <link name="laser_frame">
-        <visual>
-            <geometry>
-                <cylinder radius="0.035" length="0.04"/>
-            </geometry>
-            <material name="black"/>
-        </visual>
-        <collision>
-            <geometry>
-                <cylinder radius="0.035" length="0.04"/>
-            </geometry>
-        </collision>
-        <xacro:inertial_cylinder mass="0.1" length="0.04" radius="0.035">
-            <origin xyz = "0 0 0" rpy = "0 0 0 "/>
-        </xacro:inertial_cylinder>
-    </link>
-     <gazebo reference="laser_frame">
-        <material>Gazebo/Black</material>
-        <sensor name="laser" type="ray">
-            <pose> 0 0 0 0 0 0 </pose>
-            <visualize>true</visualize>
-            <update_rate>10</update_rate>
-            <ray>
-                <scan>
-                    <horizontal>
-                        <samples>360</samples>
-                        <min_angle>-3.14</min_angle>
-                        <max_angle>3.14</max_angle>
-                    </horizontal>
-                </scan>
-                <range>
-                    <min>0.3</min>
-                    <max>12</max>
-                </range>
-            </ray>
-            <plugin name="laser_controller" filename="libgazebo_ros_ray_sensor.so">
-                <ros>
-                    <argument>~/out:=scan</argument>
-                </ros>
-                <output_type>sensor_msgs/LaserScan</output_type>
-                <frame_name>laser_frame</frame_name>
-            </plugin>
-        </sensor>
-    </gazebo>
+<robot xmlns:xacro="http://www.ros.org/wiki/xacro">
+  <!-- Define your robot's transmission, joints, and other components here -->
+  <!-- Define the lidar joint -->
+  <joint name="lidar_joint" type="fixed">
+    <parent link="chassis"/>
+    <child link="lidar_frame"/>
+    <origin xyz="0.87 0 0.38" rpy="0 0 0"/>
+  </joint>
+  <!-- Define the lidar frame link -->
+  <link name="lidar_frame">
+    <visual>
+      <geometry>
+        <cylinder radius="0.035" length="0.04"/>
+      </geometry>
+      <material name="Gazebo/Black"/> <!-- Updated material name -->
+    </visual>
+    <collision>
+      <geometry>
+        <cylinder radius="0.035" length="0.04"/>
+      </geometry>
+    </collision>
+    <inertial>
+      <mass value="0.1"/>
+      <inertia ixx="0.0" ixy="0.0" ixz="0.0" iyy="0.0" iyz="0.0" izz="0.0"/>
+    </inertial>
+  </link>
+  <!-- Define the lidar sensor in Gazebo -->
+  <gazebo reference="lidar_frame">
+    <material>Gazebo/Black</material>
+    <!-- Define the lidar sensor -->
+    <sensor name="lidar" type="gpu_ray" always_on="true">
+      <pose>0 0 0 0 0 0</pose>
+      <visualize>true</visualize>
+      <update_rate>10</update_rate>
+      <ray>
+        <scan>
+          <horizontal>
+            <samples>360</samples>
+            <min_angle>-3.14</min_angle>
+            <max_angle>3.14</max_angle>
+          </horizontal>
+          <vertical>
+            <samples>16</samples>
+            <min_angle>-0.5</min_angle>
+            <max_angle>0.5</max_angle>
+          </vertical>
+        </scan>
+        <range>
+          <min>0.3</min>
+          <max>12</max>
+        </range>
+      </ray>
+      <!-- Use <gazebo_ros> tag to specify Gazebo ROS plugin -->
+      <plugin name="lidar_controller" filename="libgazebo_ros_gpu_laser.so">
+        <ros>
+          <arguments>
+            <!-- Use <param> to specify parameters for the plugin -->
+            <param name="frame_name" value="lidar_frame"/>
+            <param name="output_topic" value="scan"/>
+          </arguments>
+        </ros>
+        <output_type>sensor_msgs/LaserScan</output_type>
+      </plugin>
+    </sensor>
+  </gazebo>
 </robot>

File: install/model_py/share/model_py/urdf/run.urdf.xacro (robot description, xacro)
@@ -5,5 +5,6 @@
     <xacro:include filename="gazebo_control.xacro" />
     <!-- <xacro:include filename="lidar.urdf.xacro" /> -->
-    <xacro:include filename="ir.urdf.xacro" />
+    <!-- <xacro:include filename="ir.urdf.xacro" /> -->
+    <xacro:include filename="lidar3d.urdf.xacro" />
     <!-- <xacro:if value="$(arg use_ros2_control)">
         <xacro:include filename="ros2_control.xacro" />
@@ -14,5 +15,5 @@
     <xacro:include filename="lidar.xacro" />
     <<xacro:include filename="camera.xacro" /> -->
-    <!-- <xacro:include filename="depth_camera.xacro" />  -->
+    <!-- <xacro:include filename="depthcamera.urdf.xacro" />  -->
     <!-- <xacro:include filename="face.xacro" /> -->
 </robot>

Commit message: commit_these

File: install/model_py/share/model_py/urdf/lidar.urdf.xacro (robot description, xacro)
@@ -1,67 +1,53 @@
 <?xml version="1.0"?>
-<robot xmlns:xacro="http://www.ros.org/wiki/xacro">
-  <!-- Define your robot's transmission, joints, and other components here -->
-  <!-- Define the lidar joint -->
-  <joint name="lidar_joint" type="fixed">
-    <parent link="chassis"/>
-    <child link="lidar_frame"/>
-    <origin xyz="0.87 0 0.38" rpy="0 0 0"/>
-  </joint>
-  <!-- Define the lidar frame link -->
-  <link name="lidar_frame">
-    <visual>
-      <geometry>
-        <cylinder radius="0.035" length="0.04"/>
-      </geometry>
-      <material name="Gazebo/Black"/> <!-- Updated material name -->
-    </visual>
-    <collision>
-      <geometry>
-        <cylinder radius="0.035" length="0.04"/>
-      </geometry>
-    </collision>
-    <inertial>
-      <mass value="0.1"/>
-      <inertia ixx="0.0" ixy="0.0" ixz="0.0" iyy="0.0" iyz="0.0" izz="0.0"/>
-    </inertial>
-  </link>
-  <!-- Define the lidar sensor in Gazebo -->
-  <gazebo reference="lidar_frame">
-    <material>Gazebo/Black</material>
-    <!-- Define the lidar sensor -->
-    <sensor name="lidar" type="gpu_ray" always_on="true">
-      <pose>0 0 0 0 0 0</pose>
-      <visualize>true</visualize>
-      <update_rate>10</update_rate>
-      <ray>
-        <scan>
-          <horizontal>
-            <samples>360</samples>
-            <min_angle>-3.14</min_angle>
-            <max_angle>3.14</max_angle>
-          </horizontal>
-          <vertical>
-            <samples>16</samples>
-            <min_angle>-0.5</min_angle>
-            <max_angle>0.5</max_angle>
-          </vertical>
-        </scan>
-        <range>
-          <min>0.3</min>
-          <max>12</max>
-        </range>
-      </ray>
-      <!-- Use <gazebo_ros> tag to specify Gazebo ROS plugin -->
-      <plugin name="lidar_controller" filename="libgazebo_ros_gpu_laser.so">
-        <ros>
-          <arguments>
-            <!-- Use <param> to specify parameters for the plugin -->
-            <param name="frame_name" value="lidar_frame"/>
-            <param name="output_topic" value="scan"/>
-          </arguments>
-        </ros>
-        <output_type>sensor_msgs/LaserScan</output_type>
-      </plugin>
-    </sensor>
-  </gazebo>
+<robot xmlns:xacro="http://www.ros.org/wiki/xacro" >
+    <joint name="laser_joint" type="fixed">
+        <parent link="chassis"/>
+        <child link="laser_frame"/>
+        <origin xyz="0.215 0 0.11" rpy="0 0 0"/>
+    </joint>
+    <link name="laser_frame">
+        <visual>
+            <geometry>
+                <cylinder radius="0.035" length="0.04"/>
+            </geometry>
+            <material name="black"/>
+        </visual>
+        <collision>
+            <geometry>
+                <cylinder radius="0.035" length="0.04"/>
+            </geometry>
+        </collision>
+        <xacro:inertial_cylinder mass="0.1" length="0.04" radius="0.035">
+            <origin xyz = "0 0 0" rpy = "0 0 0 "/>
+        </xacro:inertial_cylinder>
+    </link>
+     <gazebo reference="laser_frame">
+        <material>Gazebo/Black</material>
+        <sensor name="laser" type="ray">
+            <pose> 0 0 0 0 0 0 </pose>
+            <visualize>true</visualize>
+            <update_rate>10</update_rate>
+            <ray>
+                <scan>
+                    <horizontal>
+                        <samples>360</samples>
+                        <min_angle>-3.14</min_angle>
+                        <max_angle>3.14</max_angle>
+                    </horizontal>
+                </scan>
+                <range>
+                    <min>0.3</min>
+                    <max>12</max>
+                </range>
+            </ray>
+            <plugin name="laser_controller"
+            filename="libgazebo_ros_ray_sensor.so">
+                <ros>
+                    <argument>~/out:=scan</argument>
+                </ros>
+                <output_type>sensor_msgs/LaserScan</output_type>
+                <frame_name>laser_frame</frame_name>
+            </plugin>
+        </sensor>
+    </gazebo>
 </robot>

File: install/model_py/share/model_py/urdf/lidar3d.urdf.xacro (robot description, xacro)
@@ -22,5 +22,5 @@
     </collision>
     <inertial>
-      <mass value="0.1"/>
+      <mass value="0.0"/>
       <inertia ixx="0.0" ixy="0.0" ixz="0.0" iyy="0.0" iyz="0.0" izz="0.0"/>
     </inertial>
@@ -53,13 +53,11 @@
       </ray>
       <!-- Use <gazebo_ros> tag to specify Gazebo ROS plugin -->
-      <plugin name="lidar_controller" filename="libgazebo_ros_gpu_laser.so">
-        <ros>
-          <arguments>
-            <!-- Use <param> to specify parameters for the plugin -->
-            <param name="frame_name" value="lidar_frame"/>
-            <param name="output_topic" value="scan"/>
-          </arguments>
+        <plugin name="laser_controller"
+        filename="libgazebo_ros_ray_sensor.so">
+          <ros>
+            <argument>~/out:=scan</argument>
         </ros>
         <output_type>sensor_msgs/LaserScan</output_type>
+        <frame_name>laser_frame</frame_name>
       </plugin>
     </sensor>

File: install/model_py/share/model_py/urdf/run.urdf.xacro (robot description, xacro)
@@ -4,7 +4,9 @@
     <xacro:include filename="robot_core.urdf.xacro" />
     <xacro:include filename="gazebo_control.xacro" />
+    <xacro:include filename="depthcamera.urdf.xacro" />
+    <!-- <xacro:include filename="th3lidar.urdf.xacro" /> -->
     <!-- <xacro:include filename="lidar.urdf.xacro" /> -->
     <!-- <xacro:include filename="ir.urdf.xacro" /> -->
-    <xacro:include filename="lidar3d.urdf.xacro" />
+    <!-- <xacro:include filename="lidar3d.urdf.xacro" /> -->
     <!-- <xacro:if value="$(arg use_ros2_control)">
         <xacro:include filename="ros2_control.xacro" />

File: src/model_py/urdf/lidar.urdf.xacro (robot description, xacro)
@@ -41,5 +41,6 @@
                 </range>
             </ray>
-            <plugin name="laser_controller" filename="libgazebo_ros_ray_sensor.so">
+            <plugin name="laser_controller"
+            filename="libgazebo_ros_ray_sensor.so">
                 <ros>
                     <argument>~/out:=scan</argument>
