Commit message: commit

File: install/model_py/share/model_py/urdf/depthcamera.urdf.xacro (robot description, xacro)
@@ -4,5 +4,5 @@
         <parent link="chassis"/>
         <child link="camera_link"/>
-        <origin xyz="0.9 0 0.25" rpy="0 0 0"/>
+        <origin xyz="0.9 0.3 0.25" rpy="0 ${pi/6} 0"/>
     </joint>
     <link name="camera_link">

File: install/model_py/share/model_py/urdf/gazebo_control.xacro (robot description, xacro)
@@ -10,5 +10,5 @@
         <!--limits-->
         <max_wheel_torque>150</max_wheel_torque>
-        <max_wheel_accleration>2.0</max_wheel_accleration>
+        <max_wheel_accleration>4.0</max_wheel_accleration>
         <!--Output-->
         <odometry_frame>odom</odometry_frame>

File: install/model_py/share/model_py/urdf/lidar.urdf.xacro (robot description, xacro)
@@ -4,10 +4,10 @@
         <parent link="chassis"/>
         <child link="laser_frame"/>
-        <origin xyz="0.215 0 0.11" rpy="0 0 0"/>
+        <origin xyz="0.8 0 0.38" rpy="0 0 0"/>
     </joint>
     <link name="laser_frame">
         <visual>
             <geometry>
-                <cylinder radius="0.035" length="0.04"/>
+                <cylinder radius="0.075" length="0.04"/>
             </geometry>
             <material name="black"/>

File: install/model_py/share/model_py/urdf/robot_core.urdf.xacro (robot description, xacro)
@@ -56,5 +56,5 @@
         <parent link="base_link"/>
         <child link="left_wheel"/>
-        <origin xyz="0.3 0.4 -0.25" rpy="-${pi/2} 0 0"/>  <!-- we are rotating the whole bot 90 degrees wrt x axis..-->
+        <origin xyz="-0.5 0.4 -0.25" rpy="-${pi/2} 0 0"/>  <!-- we are rotating the whole bot 90 degrees wrt x axis..-->
         <axis xyz="0 0 1"/>
     </joint>
@@ -62,5 +62,5 @@
         <visual>
             <geometry>
-                <cylinder radius="0.25" length="0.130"/>
+                <cylinder radius="0.15" length="0.130"/>
             </geometry>
             <material name="black"/>
@@ -68,5 +68,5 @@
         <collision>
             <geometry>
-                <sphere radius="0.25"/>
+                <sphere radius="0.15"/>
             </geometry>
         </collision>
@@ -82,5 +82,5 @@
         <parent link="base_link"/>
         <child link="right_wheel"/>
-        <origin xyz="0.3 -0.4 -0.25" rpy="${pi/2} 0 0"/>  <!-- we are rotating the whole bot 90 degrees wrt x axis..-->
+        <origin xyz="-0.5 -0.4 -0.25" rpy="${pi/2} 0 0"/>  <!-- we are rotating the whole bot 90 degrees wrt x axis..-->
         <axis xyz="0 0 -1"/>
     </joint>
@@ -88,5 +88,5 @@
         <visual>
             <geometry>
-                <cylinder radius="0.25" length="0.130"/>
+                <cylinder radius="0.15" length="0.130"/>
             </geometry>
             <material name="black"/>
@@ -94,5 +94,5 @@
         <collision>
             <geometry>
-                <sphere radius="0.25"/>
+                <sphere radius="0.15"/>
             </geometry>
             <material name="black"/>
@@ -109,10 +109,10 @@
         <parent link="chassis"/>
         <child link="caster_wheel_left"/>
-        <origin xyz="-0.35 0 -0.3"/>
+        <origin xyz="0.65 0 -0.3"/>
     </joint>
     <link name="caster_wheel_left">
         <visual>
             <geometry>
-                <sphere radius="0.2"/>
+                <sphere radius="0.1"/>
             </geometry>
             <material name="black"/>
@@ -120,5 +120,5 @@
         <collision>
             <geometry>
-                <sphere radius="0.2"/>
+                <sphere radius="0.1"/>
             </geometry>
             <material name="black"/>

File: install/model_py/share/model_py/urdf/run.urdf.xacro (robot description, xacro)
@@ -5,7 +5,8 @@
     <xacro:include filename="gazebo_control.xacro" />
     <xacro:include filename="depthcamera.urdf.xacro" />
+    <xacro:include filename="depthcam2.urdf.xacro" />
     <!-- <xacro:include filename="th3lidar.urdf.xacro" /> -->
     <!-- <xacro:include filename="lidar.urdf.xacro" /> -->
-    <!-- <xacro:include filename="ir.urdf.xacro" /> -->
+    <!-- <xacro:include filename="imu.urdf.xacro" /> -->
     <!-- <xacro:include filename="lidar3d.urdf.xacro" /> -->
     <!-- <xacro:if value="$(arg use_ros2_control)">
